Commit message: Modified robot urdf.

File: 6_HCSR04/ros2_ws/src/droid1/urdf/ddd.urdf (robot description, URDF)
Before this commit: robot DDD, 10 links, 9 joints
Links:
- removed link range_back
- removed link range_front
Joints:
- removed joint hassis_to_range_back
- removed joint motor_chassis_to_range_front

Commit message: Added changes to ros2 environment- urdf, package, launch files; not sure of them lol

File: 6_HCSR04/ros2_ws/src/droid1/urdf/ddd.urdf (robot description, URDF)
Before this commit: robot DDD, 8 links, 7 joints
Links:
- removed link lidar
- removed link motor_chassis
- removed link wheel_center
- removed link wheel_left
- removed link wheel_right
- added link camera_link; visual box size=0.010 0.03 0.03
- added link camera_link_optical
- added link laser; visual cylinder length=0.04 radius=0.05
- added link wheel_back_left; visual cylinder length=0.055 radius=0.065
- added link wheel_back_right; visual cylinder length=0.055 radius=0.065
- added link wheel_front_left; visual cylinder length=0.055 radius=0.065
- added link wheel_front_right; visual cylinder length=0.055 radius=0.065
- link base_link: geometry visual cylinder length=0.1 radius=0.1
- link chassis: geometry visual box size=0.290 0.185 0.004
Joints:
- removed joint chassis_to_centre
- removed joint chassis_to_motor_chassis
- added joint chassis_to_camera_link: type fixed, parent chassis, child camera_link, origin xyz=0.065 0.0 0.09 rpy=0 0 0
- added joint chassis_to_camera_link_optical: type fixed, parent camera_link, child camera_link_optical, origin xyz=0.0 0.0 0.0 rpy=${-pi/2} 0 ${-pi/2}
- added joint motor_2: type continuous, parent base_link, child wheel_back_right, origin xyz=-0.120 -0.140 0.0 rpy=1.57 0 0, axis 0 0 1
- added joint motor_3: type continuous, parent base_link, child wheel_back_left, origin xyz=-0.120 0.140 0.0 rpy=1.57 0 0, axis 0 0 -1
- joint base_to_chassis: origin xyz=0 0 0.125 rpy=0 0 ${pi/2} -> xyz=0 0 0.125 rpy=0 0 0
- joint chassis_to_lidar: child lidar -> laser; origin xyz=0.00 -0.065 0.09 rpy=0 0 ${pi/2} -> xyz=-0.065 0.0 0.09 rpy=0 0 0
- joint motor_0: axis 1 0 0 -> 0 0 1; child wheel_left -> wheel_front_right; origin xyz=${0.204/-2} 0.00 -0.060 -> xyz=0.120 -0.140 0.0 rpy=1.57 0 0; parent motor_chassis -> base_link
- joint motor_1: axis 1 0 0 -> 0 0 -1; child wheel_right -> wheel_front_left; origin xyz=${0.204/2} 0.00 -0.060 rpy=0 0 ${pi} -> xyz=0.120 0.140 0.0 rpy=1.57 0 0; parent motor_chassis -> base_link
