Commit message: modified dimensions of the camera link

File: 6_HCSR04/ros2_ws/src/droid1/urdf/AM_camera.xacro (robot description, xacro)
@@ -13,5 +13,5 @@
         <parent link="chassis"/>
         <child link="camera_link"/>
-        <origin xyz="0.065 0.0 0.09" rpy="0 0 0"/>
+        <origin xyz="0.095 0.0 0.065" rpy="0 0 0"/>
     </joint>
     <link name="camera_link_optical">
